Commit message: fix: derive steps per meter from the wheel radius

File: description/talos.urdf.xacro (robot description, xacro)
@@ -18,5 +18,5 @@
   <xacro:property name="base" value="${cfg['base']}"/>
   <!-- Named parameters shared with #60 and the controllers. -->
-  <xacro:property name="r" value="${model['wheel_radius_m']}"/>
+  <xacro:property name="r" value="${base['wheel_radius_m']}"/>
   <xacro:property name="l" value="${model['leg_length_m']}"/>
   <xacro:property name="track" value="${base['track_width_m']}"/>

Commit message: fix: derive leg length from the wheelbase and require base for model

File: description/talos.urdf.xacro (robot description, xacro)
@@ -19,5 +19,5 @@
   <!-- Named parameters shared with #60 and the controllers. -->
   <xacro:property name="r" value="${base['wheel_radius_m']}"/>
-  <xacro:property name="l" value="${model['leg_length_m']}"/>
+  <xacro:property name="l" value="${base['wheelbase_m'] / 2}"/>
   <xacro:property name="track" value="${base['track_width_m']}"/>
   <!-- bend is the hinge opening angle alpha: pi flat, bend_min at max

Commit message: fix: take the hinge joint name from config

File: description/talos.urdf.xacro (robot description, xacro)
@@ -23,4 +23,5 @@
   <!-- bend is the hinge opening angle alpha: pi flat, bend_min at max
        fold. -->
+  <xacro:property name="hinge" value="${model['hinge_joint']}"/>
   <xacro:property name="bend_min" value="${radians(model['bend_min_deg'])}"/>
   <xacro:property name="bend_max" value="${radians(model['bend_max_deg'])}"/>
@@ -66,5 +67,5 @@
        follow through their mimic joints. -->
   <link name="bend_link"/>
-  <joint name="bend" type="revolute">
+  <joint name="${hinge}" type="revolute">
     <parent link="base_link"/>
     <child link="bend_link"/>
@@ -94,5 +95,5 @@
                           sign * (pi - bend_max) / 2)}"
              effort="${bend_effort}" velocity="${bend_velocity}"/>
-      <mimic joint="bend" multiplier="${-sign / 2}"
+      <mimic joint="${hinge}" multiplier="${-sign / 2}"
              offset="${sign * pi / 2}"/>
     </joint>
@@ -169,5 +170,5 @@
          read the open point on unclaimed position joints in
          docs/ros2_control.md: the plugin would otherwise command 0 rad. -->
-    <joint name="bend">
+    <joint name="${hinge}">
       <command_interface name="position"/>
       <state_interface name="position"/>
@@ -180,5 +181,5 @@
       <plugin>transmission_interface/SimpleTransmission</plugin>
       <actuator name="bend_servo" role="actuator1"/>
-      <joint name="bend" role="joint1">
+      <joint name="${hinge}" role="joint1">
         <mechanical_reduction>${bend_reduction}</mechanical_reduction>
       </joint>

Commit message: fix: keep bend out of ros2_control until the hardware interface converts it

File: description/talos.urdf.xacro (robot description, xacro)
@@ -26,8 +26,4 @@
   <xacro:property name="bend_min" value="${radians(model['bend_min_deg'])}"/>
   <xacro:property name="bend_max" value="${radians(model['bend_max_deg'])}"/>
-  <!-- Servo radians per radian of alpha. Each leg gear turns
-       leg_gear_ratio times the servo and both legs move. -->
-  <xacro:property name="bend_reduction"
-                  value="${1 / (2 * model['leg_gear_ratio'])}"/>
   <!-- Rough STS3215 figures: 2.9 N m stall, about 4.6 rad/s. -->
   <xacro:property name="bend_effort" value="2.9"/>
@@ -167,22 +163,9 @@
     <xacro:wheel_interfaces name="${wheels[2]}"/>
     <xacro:wheel_interfaces name="${wheels[3]}"/>
-    <!-- Position in hinge radians (alpha). Before #85 starts this joint,
-         read the open point on unclaimed position joints in
-         docs/ros2_control.md: the plugin would otherwise command 0 rad. -->
-    <joint name="${hinge}">
-      <command_interface name="position"/>
-      <state_interface name="position"/>
-      <state_interface name="velocity"/>
-      <state_interface name="effort"/>
-    </joint>
-    <!-- Servo angle = alpha * bend_reduction. The topic based plugin does
-         not apply transmissions, so the bridge converts (#63, #85). -->
-    <transmission name="bend_transmission">
-      <plugin>transmission_interface/SimpleTransmission</plugin>
-      <actuator name="bend_servo" role="actuator1"/>
-      <joint name="${hinge}" role="joint1">
-        <mechanical_reduction>${bend_reduction}</mechanical_reduction>
-      </joint>
-    </transmission>
+    <!-- The hinge is left out on purpose until #85. The bridge only knows
+         enabled joints and would drop every command naming it, and nothing
+         maps alpha to the servo yet. #85 adds it back with an initial_value,
+         the alpha to servo conversion (talos_servo.model) and the flat
+         offset calibrated in #84. See docs/ros2_control.md. -->
   </ros2_control>
 </robot>

Commit message: feat: add the bend hinge to ros2_control with a launch for the whole robot

File: description/talos.urdf.xacro (robot description, xacro)
@@ -139,6 +139,6 @@
     <origin xyz="0 0 0" rpy="0 ${-pi / 2} 0"/>
   </joint>
-  <!-- Hardware: the topic based plugin and our bridge node, see
-       docs/ros2_control.md. The hardware interface itself is #85. -->
+  <!-- Hardware: the topic based plugin and our bridge node (#85), see
+       docs/ros2_control.md. -->
   <ros2_control name="talos_servo_bus" type="system">
     <hardware>
@@ -163,9 +163,20 @@
     <xacro:wheel_interfaces name="${wheels[2]}"/>
     <xacro:wheel_interfaces name="${wheels[3]}"/>
-    <!-- The hinge is left out on purpose until #85. The bridge only knows
-         enabled joints and would drop every command naming it, and nothing
-         maps alpha to the servo yet. #85 adds it back with an initial_value,
-         the alpha to servo conversion (talos_servo.model) and the flat
-         offset calibrated in #84. See docs/ros2_control.md. -->
+    <!-- The hinge in alpha (rad, pi flat). The plugin takes the state
+         interface initial_value as the first command too, sends it until a
+         controller writes a goal, and the bridge ignores goals equal
+         to it (HINGE_INITIAL_RAD in hardware_bridge_node.py), so starting
+         never moves the hinge. No <transmission>: the plugin ignores them,
+         so the bridge converts alpha to servo steps (talos_servo.hinge). -->
+    <joint name="${hinge}">
+      <command_interface name="position">
+        <param name="initial_value">${pi}</param>
+      </command_interface>
+      <state_interface name="position">
+        <param name="initial_value">${pi}</param>
+      </state_interface>
+      <state_interface name="velocity"/>
+      <state_interface name="effort"/>
+    </joint>
   </ros2_control>
 </robot>

Commit message: fix: keep a disabled hinge out of ros2_control so the wheels still run

File: description/talos.urdf.xacro (robot description, xacro)
@@ -24,4 +24,8 @@
        fold. -->
   <xacro:property name="hinge" value="${model['hinge_joint']}"/>
+  <!-- A disabled hinge stays out of <ros2_control>: the bridge rejects a
+       whole command that names a joint it does not drive. -->
+  <xacro:property name="hinge_enabled"
+                  value="${cfg['joints'][hinge].get('enabled', True)}"/>
   <xacro:property name="bend_min" value="${radians(model['bend_min_deg'])}"/>
   <xacro:property name="bend_max" value="${radians(model['bend_max_deg'])}"/>
@@ -169,14 +173,16 @@
          <transmission>: the plugin ignores them, so the bridge converts
          alpha to servo steps (talos_servo.hinge). -->
-    <joint name="${hinge}">
-      <command_interface name="position">
-        <param name="initial_value">${pi}</param>
-      </command_interface>
-      <state_interface name="position">
-        <param name="initial_value">${pi}</param>
-      </state_interface>
-      <state_interface name="velocity"/>
-      <state_interface name="effort"/>
-    </joint>
+    <xacro:if value="${hinge_enabled}">
+      <joint name="${hinge}">
+        <command_interface name="position">
+          <param name="initial_value">${pi}</param>
+        </command_interface>
+        <state_interface name="position">
+          <param name="initial_value">${pi}</param>
+        </state_interface>
+        <state_interface name="velocity"/>
+        <state_interface name="effort"/>
+      </joint>
+    </xacro:if>
   </ros2_control>
 </robot>

Commit message: feat: feetech hardware interface with the bend hinge in ros2_control (#109)
* feat: convert the hinge opening angle to bend servo steps

* feat: add the bend hinge to ros2_control with a launch for the whole robot

* feat: drive the hinge in alpha from the hardware bridge and ignore the startup goal

* docs: describe the hinge interfaces and the whole robot bench check

* fix: require the fixed hinge flat position and clamp bend to the hinge range

* fix: arm position joints on a new goal and report an unknown hinge angle as nan

* docs: describe the fixed hinge flat position and the startup guard

* refactor: share the inverted position helper and build the hinge once on load

* fix: rearm the hinge after quiet commands and drop goals while its reading is unknown

* fix: keep a disabled hinge out of ros2_control so the wheels still run

* docs: describe the hinge rearm, dropped goals and disabled hinge

* fix: put the hinge flat position at step 4000 to leave a margin before the wrap

File: description/talos.urdf.xacro (robot description, xacro)
@@ -24,4 +24,8 @@
        fold. -->
   <xacro:property name="hinge" value="${model['hinge_joint']}"/>
+  <!-- A disabled hinge stays out of <ros2_control>: the bridge rejects a
+       whole command that names a joint it does not drive. -->
+  <xacro:property name="hinge_enabled"
+                  value="${cfg['joints'][hinge].get('enabled', True)}"/>
   <xacro:property name="bend_min" value="${radians(model['bend_min_deg'])}"/>
   <xacro:property name="bend_max" value="${radians(model['bend_max_deg'])}"/>
@@ -139,6 +143,6 @@
     <origin xyz="0 0 0" rpy="0 ${-pi / 2} 0"/>
   </joint>
-  <!-- Hardware: the topic based plugin and our bridge node, see
-       docs/ros2_control.md. The hardware interface itself is #85. -->
+  <!-- Hardware: the topic based plugin and our bridge node (#85), see
+       docs/ros2_control.md. -->
   <ros2_control name="talos_servo_bus" type="system">
     <hardware>
@@ -163,9 +167,22 @@
     <xacro:wheel_interfaces name="${wheels[2]}"/>
     <xacro:wheel_interfaces name="${wheels[3]}"/>
-    <!-- The hinge is left out on purpose until #85. The bridge only knows
-         enabled joints and would drop every command naming it, and nothing
-         maps alpha to the servo yet. #85 adds it back with an initial_value,
-         the alpha to servo conversion (talos_servo.model) and the flat
-         offset calibrated in #84. See docs/ros2_control.md. -->
+    <!-- The hinge in alpha (rad, pi flat). The plugin takes the state
+         interface initial_value as the first command too and repeats it
+         until a controller writes a goal; the bridge ignores the first
+         goal and its repeats, so starting never moves the hinge. No
+         <transmission>: the plugin ignores them, so the bridge converts
+         alpha to servo steps (talos_servo.hinge). -->
+    <xacro:if value="${hinge_enabled}">
+      <joint name="${hinge}">
+        <command_interface name="position">
+          <param name="initial_value">${pi}</param>
+        </command_interface>
+        <state_interface name="position">
+          <param name="initial_value">${pi}</param>
+        </state_interface>
+        <state_interface name="velocity"/>
+        <state_interface name="effort"/>
+      </joint>
+    </xacro:if>
   </ros2_control>
 </robot>

Commit message: fix: add the camera optical frame to the robot model

File: description/talos.urdf.xacro (robot description, xacro)
@@ -143,4 +143,12 @@
     <origin xyz="0 0 0" rpy="0 ${-pi / 2} 0"/>
   </joint>
+  <!-- Image frame for the camera node (REP 103 optical: z forward, x right,
+       y down). -->
+  <link name="camera_optical_frame"/>
+  <joint name="camera_optical_joint" type="fixed">
+    <parent link="camera_link"/>
+    <child link="camera_optical_frame"/>
+    <origin xyz="0 0 0" rpy="${-pi / 2} 0 ${-pi / 2}"/>
+  </joint>
   <!-- Hardware: the topic based plugin and our bridge node (#85), see
        docs/ros2_control.md. -->

Commit message: feat: use the calibrated max fold as the urdf bend limit

File: description/talos.urdf.xacro (robot description, xacro)
@@ -13,4 +13,7 @@
   <!-- A relative path is relative to this file. -->
   <xacro:arg name="robot_config" default="../config/robot.yaml"/>
+  <!-- Max fold from config/bend_calibration.yaml (#84), passed by the
+       launch files; empty keeps model.bend_min_deg. -->
+  <xacro:arg name="bend_min_deg" default=""/>
   <xacro:property name="cfg" lazy_eval="false"
                   value="${xacro.load_yaml('$(arg robot_config)')}"/>
@@ -28,5 +31,7 @@
   <xacro:property name="hinge_enabled"
                   value="${cfg['joints'][hinge].get('enabled', True)}"/>
-  <xacro:property name="bend_min" value="${radians(model['bend_min_deg'])}"/>
+  <xacro:property name="bend_min" value="${radians(
+      float(xacro.arg('bend_min_deg')) if xacro.arg('bend_min_deg')
+      else model['bend_min_deg'])}"/>
   <xacro:property name="bend_max" value="${radians(model['bend_max_deg'])}"/>
   <!-- Rough STS3215 figures: 2.9 N m stall, about 4.6 rad/s. -->

Commit message: feat: read the imu mount from the robot config in the urdf

File: description/talos.urdf.xacro (robot description, xacro)
@@ -133,11 +133,15 @@
   <xacro:wheel name="${wheels[3]}" leg="rear_leg" x="${-l}"
                y="${-track / 2}"/>
-  <!-- Sensors on the platform. Zero offsets until measured: #91 fills the
-       IMU, #77 the camera. -->
+  <!-- Sensors on the platform. The IMU mount comes from `imu` in the config
+       (#91); the camera offset is zero until measured (#77). -->
+  <xacro:property name="imu" value="${cfg.get('imu', dict())}"/>
+  <xacro:property name="imu_xyz" value="${imu.get('xyz', [0, 0, 0])}"/>
+  <xacro:property name="imu_rpy" value="${imu.get('rpy', [0, 0, 0])}"/>
   <link name="imu_link"/>
   <joint name="imu_joint" type="fixed">
     <parent link="base_link"/>
     <child link="imu_link"/>
-    <origin xyz="0 0 0" rpy="0 0 0"/>
+    <origin xyz="${imu_xyz[0]} ${imu_xyz[1]} ${imu_xyz[2]}"
+            rpy="${imu_rpy[0]} ${imu_rpy[1]} ${imu_rpy[2]}"/>
   </joint>
   <!-- The camera looks up at the ceiling: its x axis points along +z. -->

Commit message: feat: switch off the hinge software end stops with model.hinge_limits

File: description/talos.urdf.xacro (robot description, xacro)
@@ -34,5 +34,6 @@
       float(xacro.arg('bend_min_deg')) if xacro.arg('bend_min_deg')
       else model['bend_min_deg'])}"/>
-  <xacro:property name="bend_max" value="${radians(model['bend_max_deg'])}"/>
+  <xacro:property name="bend_max" value="${radians(model['bend_max_deg'])
+      if model.get('hinge_limits', True) else 2 * pi}"/>
   <!-- Rough STS3215 figures: 2.9 N m stall, about 4.6 rad/s. -->
   <xacro:property name="bend_effort" value="2.9"/>
